File: hardware/core/core.kicad_sch (KiCad schematic)
At the start: 0 parts

Commit message: added variables
Other:
- removed sheet sensor_board
- title: (none) -> Xihe
Changed lines of the file:
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@@
 	(generator_version "9.0")
 	(paper "A4")
+	(title_block
+		(title "Xihe")
+		(date "2025-08-19")
+		(rev "0.1")
+	)
 	(wire
 		(pts
-			(xy 114.3 76.2) (xy 127 76.2)
+			(xy 147.32 97.79) (xy 160.02 97.79)
 		)
 		(stroke
@@
 	)
 	(sheet
-		(at 88.9 63.5)
+		(at 121.92 85.09)
 		(size 25.4 25.4)
 		(exclude_from_sim no)
@@
 		)
 		(property "Sheetname" "system"
-			(at 88.9 62.7884 0)
+			(at 121.92 84.3784 0)
 			(effects
 				(font
@@
 		)
 		(property "Sheetfile" "system.kicad_sch"
-			(at 88.9 89.4846 0)
+			(at 121.92 111.0746 0)
 			(effects
 				(font
@@
 		)
 		(pin "VBAT_OK_MCU" input
-			(at 114.3 76.2 0)
+			(at 147.32 97.79 0)
 			(effects
 				(font
@@
 	)
 	(sheet
-		(at 127 63.5)
+		(at 160.02 85.09)
 		(size 25.4 25.4)
 		(exclude_from_sim no)
@@
 		)
 		(property "Sheetname" "harvester"
-			(at 127 62.7884 0)
+			(at 160.02 84.3784 0)
 			(effects
 				(font
@@
 		)
 		(property "Sheetfile" "harvester.kicad_sch"
-			(at 127 89.4846 0)
+			(at 160.02 111.0746 0)
 			(effects
 				(font
@@
 		)
 		(pin "VBAT_OK_MCU" output
-			(at 127 76.2 180)
+			(at 160.02 97.79 180)
 			(effects
 				(font
@@
 				)
 			)
-		)
-	)
-	(sheet
-		(at 88.9 101.6)
-		(size 63.5 12.7)
-		(exclude_from_sim no)
-		(in_bom yes)
-		(on_board yes)
-		(dnp no)
-		(fields_autoplaced yes)
-		(stroke
-			(width 0.1524)
-			(type solid)
-		)
-		(fill
-			(color 0 255 0 1.0000)
-		)
-		(property "Sheetname" "sensor_board"
-			(at 88.9 100.8884 0)
-			(effects
-				(font
-					(size 1.27 1.27)
-				)
-				(justify left bottom)
-			)
-		)
-		(property "Sheetfile" "sensor_board.kicad_sch"
-			(at 88.9 114.8846 0)
-			(effects
-				(font
-					(size 1.27 1.27)
-				)
-				(justify left top)
-			)
-		)
-		(instances
-			(project "core"
-				(path "/8ec7ca4f-74cd-48e1-b45d-8806dcda5073"
-					(page "4")
-				)
-			)
