File: hardware/core/core.kicad_pcb (KiCad board)
At the start: 2 copper layers, 23 x 33 mm, 29 parts, among them J1 MOLEX_SlimStack_505550-1020, J2 Conn_01x02_Pin, U1 XIAO-NRF54L15, U2 BQ25173DSG, U3 BQ25570, U5 AXP1T34

Commit message: corrections from footprint updates and manufacture file exports
Parts:
- removed U5: AXP1T34, generic:NX_6SOT1202
- added U4: AXP1T34, generic:NX_5SOT353, B.Cu at (85.6, 79.0)
- R1: value 750 -> 3k
- ROUT1, ROUT2: value 6.49 -> 6.49M
- U2: footprint generic:WSON-8-1EP_2x2mm_P0.5mm_EP0.9x1.6mm -> generic:TI_8WSON_DSG
- U3: footprint generic:QFN-20-1EP_3.5x3.5mm_P0.5mm_EP2x2mm -> generic:TI_20VQFN_RGR
Routing:
- net +3V3: track 44.6 -> 38.9 mm
- net /harvester/VBAT_OK: track 20.8 -> 20.1 mm
