File: hardware/core/harvester.kicad_sch (KiCad schematic)
At the start: 27 parts, among them J2 Conn_01x02_Pin, U2 BQ25173DSG, U3 BQ25570, U5 AXP1T34

Commit message: corrections from footprint updates and manufacture file exports
Parts:
- removed U5: AXP1T34, generic:NX_6SOT1202, symbol ic_logic:AXP1T34GSH
- added U4: AXP1T34, generic:NX_5SOT353, symbol ic_logic:AXP1T34GWH
- ROUT1, ROUT2: value 6.49 -> 6.49M
- U2: footprint generic:WSON-8-1EP_2x2mm_P0.5mm_EP0.9x1.6mm -> generic:TI_8WSON_DSG
- U3: footprint generic:QFN-20-1EP_3.5x3.5mm_P0.5mm_EP2x2mm -> generic:TI_20VQFN_RGR
Connections:
- net +3V3: now also U4.5 (VCCO)
- net GND: now also U4.3 (GND)
- net VBAT_OK: now also U4.2 (A)
- net VBAT_OK_MCU: now also U4.4 (B)
- net VCAP: now also U4.1 (VCCI)
Changed lines of the file:
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@@
 	(title_block
 		(title "Xihe")
-		(date "2025-08-28")
+		(date "2025-08-29")
 		(rev "0.1")
 	)
@@
 			)
 		)
-		(property "Value" "6.49"
+		(property "Value" "6.49M"
 			(at 80.01 64.7699 0)
 			(effects
@@
 			)
 		)
-		(property "Footprint" "generic:WSON-8-1EP_2x2mm_P0.5mm_EP0.9x1.6mm"
+		(property "Footprint" "generic:TI_8WSON_DSG"
 			(at 148.59 185.42 0)
 			(effects
@@
 	)
 	(symbol
-		(lib_id "ic_logic:AXP1T34GSH")
-		(at 243.84 53.34 0)
-		(unit 1)
-		(exclude_from_sim no)
-		(in_bom yes)
-		(on_board yes)
-		(dnp no)
-		(fields_autoplaced yes)
-		(property "Reference" "U5"
-			(at 243.84 40.64 0)
-			(effects
-				(font
-					(size 1.27 1.27)
-				)
-			)
-		)
-		(property "Value" "AXP1T34"
-			(at 243.84 43.18 0)
-			(effects
-				(font
-					(size 1.27 1.27)
-				)
-			)
-		)
-		(property "Footprint" "generic:NX_6SOT1202"
-			(at 243.84 64.77 0)
-			(effects
-				(font
-					(size 1.27 1.27)
-				)
-				(hide yes)
-			)
-		)
-		(property "Datasheet" "https://assets.nexperia.com/documents/data-sheet/AXP1T34.pdf"
-			(at 221.742 74.422 0)
-			(effects
-				(font
-					(size 1.27 1.27)
-				)
-				(hide yes)
-			)
-		)
-		(property "Description" "Dual supply unidirectional translating buffer"
-			(at 242.57 74.168 0)
-			(effects
-				(font
-					(size 1.27 1.27)
-				)
-				(hide yes)
-			)
-		)
-		(property "Part Number" "74AXP1T34GSH"
-			(at 243.84 53.34 0)
-			(effects
-				(font
-					(size 1.27 1.27)
-				)
-				(hide yes)
-			)
-		)
-		(property "Manufacturer" "Nexperia USA Inc."
-			(at 243.84 53.34 0)
-			(effects
-				(font
-					(size 1.27 1.27)
-				)
-				(hide yes)
-			)
-		)
-		(property "Mounting Type" "smt"
-			(at 243.84 53.34 0)
-			(effects
-				(font
-					(size 1.27 1.27)
-				)
-				(hide yes)
-			)
-		)
-		(property "Package" "6XSON"
-			(at 243.84 53.34 0)
-			(effects
-				(font
-					(size 1.27 1.27)
-				)
-				(hide yes)
-			)
-		)
-		(property "Short" ""
-			(at 243.84 53.34 0)
-			(effects
-				(font
-					(size 1.27 1.27)
-				)
-				(hide yes)
-			)
-		)
-		(pin "3"
-		)
-		(pin "6"
-		)
-		(pin "4"
-		)
-		(pin "5"
-		)
-		(pin "2"
-		)
-		(pin "1"
-		)
-		(instances
-			(project ""
-				(path "/8ec7ca4f-74cd-48e1-b45d-8806dcda5073/cd3a3636-14ab-4325-9b35-d239f2fcdaad"
-					(reference "U5")
-					(unit 1)
-				)
-			)
-		)
-	)
-	(symbol
 		(lib_id "power_symbol:GND")
 		(at 60.96 97.79 0)
@@
 	)
 	(symbol
+		(lib_id "ic_logic:AXP1T34GWH")
+		(at 243.84 53.34 0)
+		(unit 1)
+		(exclude_from_sim no)
+		(in_bom yes)
+		(on_board yes)
+		(dnp no)
+		(fields_autoplaced yes)
+		(property "Reference" "U4"
+			(at 243.84 40.64 0)
+			(effects
+				(font
+					(size 1.27 1.27)
+				)
+			)
+		)
+		(property "Value" "AXP1T34"
+			(at 243.84 43.18 0)
+			(effects
+				(font
+					(size 1.27 1.27)
+				)
+			)
+		)
+		(property "Footprint" "generic:NX_5SOT353"
+			(at 243.84 64.77 0)
+			(effects
+				(font
+					(size 1.27 1.27)
+				)
+				(hide yes)
+			)
+		)
+		(property "Datasheet" "https://assets.nexperia.com/documents/data-sheet/AXP1T34.pdf"
+			(at 221.742 74.422 0)
+			(effects
+				(font
+					(size 1.27 1.27)
+				)
+				(hide yes)
+			)
+		)
+		(property "Description" "Dual supply unidirectional translating buffer"
+			(at 242.57 74.168 0)
+			(effects
+				(font
+					(size 1.27 1.27)
+				)
+				(hide yes)
+			)
+		)
+		(property "Manufacturer" "Nexperia USA Inc."
+			(at 243.84 53.34 0)
+			(effects
+				(font
+					(size 1.27 1.27)
+				)
+				(hide yes)
+			)
+		)
+		(property "Mounting Type" "smt"
+			(at 243.84 53.34 0)
+			(effects
+				(font
+					(size 1.27 1.27)
+				)
+				(hide yes)
+			)
+		)
+		(property "Part Number" "74AXP1T34GWH"
+			(at 243.84 53.34 0)
+			(effects
+				(font
+					(size 1.27 1.27)
+				)
+				(hide yes)
+			)
+		)
+		(pin "4"
+		)
+		(pin "1"
+		)
+		(pin "2"
+		)
+		(pin "3"
+		)
+		(pin "5"
+		)
+		(instances
+			(project ""
+				(path "/8ec7ca4f-74cd-48e1-b45d-8806dcda5073/cd3a3636-14ab-4325-9b35-d239f2fcdaad"
+					(reference "U4")
+					(unit 1)
+				)
+			)
+		)
+	)
+	(symbol
 		(lib_id "passive:C")
 		(at 105.41 40.64 0)
@@
 			)
 		)
-		(property "Value" "6.49"
+		(property "Value" "6.49M"
 			(at 80.01 77.4699 0)
 			(effects
@@
 			)
 		)
-		(property "Footprint" "generic:QFN-20-1EP_3.5x3.5mm_P0.5mm_EP2x2mm"
+		(property "Footprint" "generic:TI_20VQFN_RGR"
 			(at 137.16 46.99 0)
 			(effects
