File: hardware/sense_ambient/ambient.kicad_sch (KiCad schematic)
At the start: 9 parts, among them J1 MOLEX_SlimStack_505551-1020, SW1 ReedSW_NO, U1 OPT3002DNPR, U2 HDC2010YPAR

Commit message: updated technical sheet
Parts:
- SW1: footprint part_specific:COMUS_RI80SMDM0510G1 -> part_specific:COMUS_RI80SMDM0510J1; Part Number RI80SMDM-0510-G1 -> RI80SMDM-0510-J1
Changed lines of the file:
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@@
 			)
 		)
-		(property "Footprint" "part_specific:COMUS_RI80SMDM0510G1"
+		(property "Footprint" "part_specific:COMUS_RI80SMDM0510J1"
 			(at 137.16 125.73 0)
 			(effects
@@
 			)
 		)
-		(property "Part Number" "RI80SMDM-0510-G1"
+		(property "Part Number" "RI80SMDM-0510-J1"
 			(at 137.16 125.73 90)
 			(effects
