File: hardware/sense_ambient/ambient.kicad_sch (KiCad schematic)
At the start: 9 parts, among them J1 MOLEX_SlimStack_505551-1020, SW1 ReedSW_NO, U1 OPT3002DNPR, U2 HDC2010YPAR

Commit message: corrections from footprint updates and manufacture file exports
Other:
- moved on the sheet: C1, C2, J1, R1, R2, R3, SW1, U1, U2
