File: hardware/sense_ambient/ambient.kicad_pcb (KiCad board)
At the start: 2 copper layers, 12.5 x 11 mm, 9 parts, among them J1 MOLEX_SlimStack_505551-1020, SW1 ReedSW_NO, U1 OPT3002DNPR, U2 HDC2010YPAR

Commit message: corrections from footprint updates and manufacture file exports
Parts:
- moved U2 0.06 mm to (110.1, 58.8)
